Commit message: lizard-v6: rotate asset forward axis head +Y to +X
Rigid -90 deg Z rotation of the whole rig so the head sits on base +X, the frame the velocity task commands and rewards. Blend SSOT rotated via headless rotate_rig.py (1e-6 rigidity self-check; rotation kept as armature object transform because transform_apply drifts through bone-roll round-trips), generate_urdf reads world-space bone heads and carries the rotated AXIS_MAP, fix_bones converts world<->armature explicitly. URDF/STL/OBJ/USD regenerated through the full pipeline; tree-wide asset locks refreshed in the same commit (intentional retirement of the Y-axis asset).

File: rl_exp/versions/lizard/lizard.urdf (robot description, URDF)
Before this commit: robot lizard_robot, 27 links, 26 joints
Joints:
- joint lf_foot_joint: axis 1 0 0 -> 0 -1 0; origin xyz=-0.039465 0.000001 -0.124654 rpy=0 0 0 -> xyz=0.000001 0.039465 -0.124654 rpy=0 0 0
- joint lf_haa_joint: axis 0 1 0 -> 1 0 0; origin xyz=-0.321462 0.596756 -0.055889 rpy=0 0 0 -> xyz=0.596756 0.321462 -0.055889 rpy=0 0 0
- joint lf_hfe_joint: origin xyz=-0.418794 0.000000 -0.276152 rpy=0 0 0 -> xyz=0.000000 0.418794 -0.276152 rpy=0 0 0
- joint lf_kfe_joint: axis 0 1 0 -> 1 0 0; origin xyz=-0.009685 -0.000000 -0.381997 rpy=0 0 0 -> xyz=-0.000000 0.009685 -0.381997 rpy=0 0 0
- joint neck1_pitch_joint: axis 1 0 0 -> 0 -1 0; origin xyz=0.000000 0.005000 0.000000 rpy=0 0 0 -> xyz=0.005000 0.000000 0.000000 rpy=0 0 0
- joint neck1_yaw_joint: origin xyz=0.000000 1.069600 0.000000 rpy=0 0 0 -> xyz=1.069600 0.000000 0.000000 rpy=0 0 0
- joint neck2_pitch_joint: axis 1 0 0 -> 0 -1 0; origin xyz=0.000000 0.005000 0.000000 rpy=0 0 0 -> xyz=0.005000 0.000000 0.000000 rpy=0 0 0
- joint neck2_yaw_joint: origin xyz=0.005500 0.539200 0.000000 rpy=0 0 0 -> xyz=0.539200 -0.005500 0.000000 rpy=0 0 0
- joint neck3_pitch_joint: axis 1 0 0 -> 0 -1 0; origin xyz=0.000000 0.005000 0.000000 rpy=0 0 0 -> xyz=0.005000 0.000000 0.000000 rpy=0 0 0
- joint neck3_yaw_joint: origin xyz=0.000000 0.429900 0.000000 rpy=0 0 0 -> xyz=0.429900 0.000000 0.000000 rpy=0 0 0
- joint rear_pitch_joint: axis 1 0 0 -> 0 -1 0; origin xyz=0.000000 0.005000 0.000000 rpy=0 0 0 -> xyz=0.005000 0.000000 0.000000 rpy=0 0 0
- joint rf_foot_joint: axis 1 0 0 -> 0 -1 0; origin xyz=0.036816 -0.000001 -0.125462 rpy=0 0 0 -> xyz=-0.000001 -0.036816 -0.125462 rpy=0 0 0
- joint rf_haa_joint: axis 0 1 0 -> 1 0 0; origin xyz=0.335819 0.602861 -0.055928 rpy=0 0 0 -> xyz=0.602861 -0.335819 -0.055928 rpy=0 0 0
- joint rf_hfe_joint: origin xyz=0.412877 0.000000 -0.284945 rpy=0 0 0 -> xyz=0.000000 -0.412877 -0.284945 rpy=0 0 0
- joint rf_kfe_joint: axis 0 1 0 -> 1 0 0; origin xyz=0.001594 0.000000 -0.382117 rpy=0 0 0 -> xyz=0.000000 -0.001594 -0.382117 rpy=0 0 0
- joint rl_foot_joint: axis 1 0 0 -> 0 -1 0; origin xyz=-0.039465 -0.000005 -0.124654 rpy=0 0 0 -> xyz=-0.000005 0.039465 -0.124654 rpy=0 0 0
- joint rl_haa_joint: axis 0 1 0 -> 1 0 0; origin xyz=-0.363333 -0.480451 -0.055936 rpy=0 0 0 -> xyz=-0.480451 0.363333 -0.055936 rpy=0 0 0
- joint rl_hfe_joint: origin xyz=-0.418806 -0.000000 -0.276146 rpy=0 0 0 -> xyz=-0.000000 0.418806 -0.276146 rpy=0 0 0
- joint rl_kfe_joint: axis 0 1 0 -> 1 0 0; origin xyz=-0.009685 -0.000043 -0.381998 rpy=0 0 0 -> xyz=-0.000043 0.009685 -0.381998 rpy=0 0 0
- joint rr_foot_joint: axis 1 0 0 -> 0 -1 0; origin xyz=0.039465 -0.000001 -0.124654 rpy=0 0 0 -> xyz=-0.000001 -0.039465 -0.124654 rpy=0 0 0
- joint rr_haa_joint: axis 0 1 0 -> 1 0 0; origin xyz=0.359465 -0.485375 -0.055891 rpy=0 0 0 -> xyz=-0.485375 -0.359465 -0.055891 rpy=0 0 0
- joint rr_hfe_joint: origin xyz=0.418791 -0.000000 -0.276154 rpy=0 0 0 -> xyz=0.000000 -0.418791 -0.276154 rpy=0 0 0
- joint rr_kfe_joint: axis 0 1 0 -> 1 0 0; origin xyz=0.009685 -0.000000 -0.381998 rpy=0 0 0 -> xyz=-0.000000 -0.009685 -0.381998 rpy=0 0 0
- joint tail_pitch_joint: axis 1 0 0 -> 0 -1 0; origin xyz=0.000000 -0.005000 0.000000 rpy=0 0 0 -> xyz=-0.005000 -0.000000 0.000000 rpy=0 0 0
- joint tail_yaw_joint: origin xyz=0.000000 -1.261300 0.189500 rpy=0 0 0 -> xyz=-1.261300 -0.000000 0.189500 rpy=0 0 0

Commit message: lizard-v8: anatomy-correct asset (net +90 flip, rename 26 joints) + yaml migration
v6 first run walked tail-first and was retired at 8950/15000 iters: the
rig's bone names are 180 deg off the model's anatomy (the "neck1-3"
chain is the tail -- build_rig antenna_tip; the "tail_yaw/tail_pitch"
chain carries the sphere HEAD; leg names front/rear + left/right
swapped). v6 rotated the NAME-head onto task +X, i.e. the anatomical
tail, so the policy walked exactly as paid (probe: disp_head
+1.2..1.6 m per 100 steps under forward commands).

- blender/rename_flip_v8.py: +180 deg Z on the stance blend (net +90
  from pre-v6: sphere head -y -> +x, antenna tail -> -x) + rename all
  26 joints to anatomy (rear->chest, tail->neck, neck1-3->tail1-3,
  legs rl<->rf / lf<->rr), mesh parent_bone re-targeting, layout gates
- generate_urdf AXIS_MAP signs flipped for the rotation; URDF/STL/OBJ
  -> convert_urdf -> flatten rerun (2.13 MB usda, 26 joints)
- migrate_joint_names_v8.py: mechanical rename across every version
  yaml (joint_order + spine regexes rear_->chest_, tail_->tail[0-9]_);
  root/v8 joint_order = actual regenerated URDF order (export_ue
  sequence gate); export_ue name-comparison suffix bug fixed
- teacher_env_cfg spine action regex (base class) + curriculum/
  parkour snapshots synced; TEACHER_PRIVILEGED_SPEC v8 entry;
  Lizard-Rough-v8 / -Play-v8 registered; V8 runner cfg
- checks: check_joints_v8.py layout hard gates (sphere head must sit
  at +x -- the v6 lesson), teacher_smoke_v8.py green, offline suite
  10/10 PARITY_OK, locks refreshed tree-wide (--update-locks, intended
  asset retirement), UE artifacts regenerated
- v6 NOTES result backfill (retired, root cause, probe evidence);
  FAMILY version table / geometry memo / mirror-axis table updated

File: rl_exp/versions/lizard/lizard.urdf (robot description, URDF)
Before this commit: robot lizard_robot, 27 links, 26 joints
Links:
- removed link neck1_pitch
- removed link neck1_yaw
- removed link neck2_pitch
- removed link neck2_yaw
- removed link neck3_pitch
- removed link neck3_yaw
- removed link rear_pitch
- removed link rear_yaw
- removed link tail_pitch
- removed link tail_yaw
- added link chest_pitch, mass 15.7685; collision mesh filename=meshes/collision/chest_pitch_collision.obj; visual mesh filename=meshes/visual/chest_pitch_visual.obj
- added link chest_yaw, mass 0.0500
- added link neck_pitch, mass 11.0551; collision mesh filename=meshes/collision/neck_pitch_collision.obj; visual mesh filename=meshes/visual/neck_pitch_visual.obj
- added link neck_yaw, mass 0.0500
- added link tail1_pitch, mass 3.9061; collision mesh filename=meshes/collision/tail1_pitch_collision.obj; visual mesh filename=meshes/visual/tail1_pitch_visual.obj
- added link tail1_yaw, mass 0.0500
- added link tail2_pitch, mass 2.3105; collision mesh filename=meshes/collision/tail2_pitch_collision.obj; visual mesh filename=meshes/visual/tail2_pitch_visual.obj
- added link tail2_yaw, mass 0.0500
- added link tail3_pitch, mass 1.5595; collision mesh filename=meshes/collision/tail3_pitch_collision.obj; visual mesh filename=meshes/visual/tail3_pitch_visual.obj
- added link tail3_yaw, mass 0.0500
Joints:
- removed joint neck1_pitch_joint
- removed joint neck1_yaw_joint
- removed joint neck2_pitch_joint
- removed joint neck2_yaw_joint
- removed joint neck3_pitch_joint
- removed joint neck3_yaw_joint
- removed joint rear_pitch_joint
- removed joint rear_yaw_joint
- removed joint tail_pitch_joint
- removed joint tail_yaw_joint
- added joint chest_pitch_joint: type revolute, parent chest_yaw, child chest_pitch, origin xyz=-0.005000 0.000000 0.000000 rpy=0 0 0, axis 0 1 0, limit lower=-0.50 upper=0.50 effort=80 velocity=4
- added joint chest_yaw_joint: type revolute, parent base_link, child chest_yaw, origin xyz=0.000000 0.000000 0.000000 rpy=0 0 0, axis 0 0 1, limit lower=-0.60 upper=0.60 effort=80 velocity=4
- added joint neck_pitch_joint: type revolute, parent neck_yaw, child neck_pitch, origin xyz=0.005000 -0.000000 0.000000 rpy=0 0 0, axis 0 1 0, limit lower=-0.50 upper=0.50 effort=80 velocity=4
- added joint neck_yaw_joint: type revolute, parent chest_pitch, child neck_yaw, origin xyz=1.261300 -0.000000 0.189500 rpy=0 0 0, axis 0 0 1, limit lower=-0.60 upper=0.60 effort=80 velocity=4
- added joint tail1_pitch_joint: type revolute, parent tail1_yaw, child tail1_pitch, origin xyz=-0.005000 0.000000 0.000000 rpy=0 0 0, axis 0 1 0, limit lower=-0.50 upper=0.50 effort=80 velocity=4
- added joint tail1_yaw_joint: type revolute, parent base_link, child tail1_yaw, origin xyz=-1.069600 0.000000 0.000000 rpy=0 0 0, axis 0 0 1, limit lower=-0.60 upper=0.60 effort=80 velocity=4
- added joint tail2_pitch_joint: type revolute, parent tail2_yaw, child tail2_pitch, origin xyz=-0.005000 0.000000 0.000000 rpy=0 0 0, axis 0 1 0, limit lower=-0.50 upper=0.50 effort=80 velocity=4
- added joint tail2_yaw_joint: type revolute, parent tail1_pitch, child tail2_yaw, origin xyz=-0.539200 0.005500 0.000000 rpy=0 0 0, axis 0 0 1, limit lower=-0.60 upper=0.60 effort=80 velocity=4
- added joint tail3_pitch_joint: type revolute, parent tail3_yaw, child tail3_pitch, origin xyz=-0.005000 0.000000 0.000000 rpy=0 0 0, axis 0 1 0, limit lower=-0.50 upper=0.50 effort=80 velocity=4
- added joint tail3_yaw_joint: type revolute, parent tail2_pitch, child tail3_yaw, origin xyz=-0.429900 0.000000 0.000000 rpy=0 0 0, axis 0 0 1, limit lower=-0.60 upper=0.60 effort=80 velocity=4
- joint lf_foot_joint: axis 0 -1 0 -> 0 1 0
- joint lf_haa_joint: axis 1 0 0 -> -1 0 0; origin xyz=0.596756 0.321462 -0.055889 rpy=0 0 0 -> xyz=0.485375 0.359465 -0.055891 rpy=0 0 0; parent base_link -> chest_pitch
- joint lf_hfe_joint: origin xyz=0.000000 0.418794 -0.276152 rpy=0 0 0 -> xyz=0.000000 0.418791 -0.276154 rpy=0 0 0
- joint lf_kfe_joint: axis 1 0 0 -> -1 0 0; origin xyz=-0.000000 0.009685 -0.381997 rpy=0 0 0 -> xyz=0.000000 0.009685 -0.381998 rpy=0 0 0
- joint rf_foot_joint: axis 0 -1 0 -> 0 1 0; origin xyz=-0.000001 -0.036816 -0.125462 rpy=0 0 0 -> xyz=0.000005 -0.039465 -0.124654 rpy=0 0 0
- joint rf_haa_joint: axis 1 0 0 -> -1 0 0; origin xyz=0.602861 -0.335819 -0.055928 rpy=0 0 0 -> xyz=0.480451 -0.363333 -0.055936 rpy=0 0 0; parent base_link -> chest_pitch
- joint rf_hfe_joint: origin xyz=0.000000 -0.412877 -0.284945 rpy=0 0 0 -> xyz=0.000000 -0.418806 -0.276146 rpy=0 0 0
- joint rf_kfe_joint: axis 1 0 0 -> -1 0 0; origin xyz=0.000000 -0.001594 -0.382117 rpy=0 0 0 -> xyz=0.000043 -0.009685 -0.381998 rpy=0 0 0
- joint rl_foot_joint: axis 0 -1 0 -> 0 1 0; origin xyz=-0.000005 0.039465 -0.124654 rpy=0 0 0 -> xyz=0.000001 0.036816 -0.125462 rpy=0 0 0
- joint rl_haa_joint: axis 1 0 0 -> -1 0 0; origin xyz=-0.480451 0.363333 -0.055936 rpy=0 0 0 -> xyz=-0.602861 0.335819 -0.055928 rpy=0 0 0; parent rear_pitch -> base_link
- joint rl_hfe_joint: origin xyz=-0.000000 0.418806 -0.276146 rpy=0 0 0 -> xyz=0.000000 0.412877 -0.284945 rpy=0 0 0
- joint rl_kfe_joint: axis 1 0 0 -> -1 0 0; origin xyz=-0.000043 0.009685 -0.381998 rpy=0 0 0 -> xyz=0.000000 0.001594 -0.382117 rpy=0 0 0
- joint rr_foot_joint: axis 0 -1 0 -> 0 1 0
- joint rr_haa_joint: axis 1 0 0 -> -1 0 0; origin xyz=-0.485375 -0.359465 -0.055891 rpy=0 0 0 -> xyz=-0.596756 -0.321462 -0.055889 rpy=0 0 0; parent rear_pitch -> base_link
- joint rr_hfe_joint: origin xyz=0.000000 -0.418791 -0.276154 rpy=0 0 0 -> xyz=0.000000 -0.418794 -0.276152 rpy=0 0 0
- joint rr_kfe_joint: axis 1 0 0 -> -1 0 0; origin xyz=-0.000000 -0.009685 -0.381998 rpy=0 0 0 -> xyz=0.000000 -0.009685 -0.381997 rpy=0 0 0
